File: esp07-breakout.kicad_pcb (KiCad board)
At the start: 2 copper layers, 40 x 40 mm, 12 parts, among them J1 Module port, SW1 FLASH, U1 ESP-07, U2 LD1117S33TR_SOT223

Commit message: Added back layer silkscreen (fixes #1); Added photo
Other:
- board text added: "+5V"
- board text added: "ADC"
- board text added: "GND"
- board text added: "GPIO0"
- board text added: "GPIO1"
- board text added: "GPIO12"
- board text added: "GPIO13"
- board text added: "GPIO14"
- board text added: "GPIO15"
- board text added: "GPIO16"
- board text added: "GPIO2"
- board text added: "GPIO3"
- board text added: "GPIO4"
- board text added: "GPIO5"
